Commit message: add lidar to laikago

File: robots/laikago_description/xacro/gazebo.xacro (robot description, xacro)
@@ -11,5 +11,6 @@
     <gazebo>
         <plugin name="3dplot" filename="libLinkPlot3DPlugin.so">
-            <frequency>10</frequency>
+            <frequency>
+                10</frequency>
             <plot>
                 <link>base</link>
@@ -32,5 +33,6 @@
     <gazebo>
         <plugin filename="libgazebo_ros_force.so" name="gazebo_ros_force">
-            <bodyName>trunk</bodyName>
+            <bodyName>
+                trunk</bodyName>
             <topicName>/apply_force/trunk</topicName>
         </plugin>
@@ -39,5 +41,6 @@
         <gravity>true</gravity>
         <sensor name="imu_sensor" type="imu">
-            <always_on>true</always_on>
+            <always_on>
+                true</always_on>
             <update_rate>1000</update_rate>
             <visualize>true</visualize>
@@ -45,12 +48,46 @@
             <plugin filename="libgazebo_ros_imu_sensor.so" name="imu_plugin">
                 <topicName>trunk_imu</topicName>
-                <bodyName>imu_link</bodyName>
+                <bodyName>
+                    imu_link</bodyName>
                 <updateRateHZ>1000.0</updateRateHZ>
                 <gaussianNoise>0.0</gaussianNoise>
                 <xyzOffset>0 0 0</xyzOffset>
-                <rpyOffset>0 0 0</rpyOffset>
+                <rpyOffset>0 0
+                    0</rpyOffset>
                 <frameName>imu_link</frameName>
             </plugin>
             <pose>0 0 0 0 0 0</pose>
+        </sensor>
+    </gazebo>
+    <gazebo reference="lidar_link">
+        <sensor name="laser" type="ray">
+            <ray>
+                <scan>
+                    <horizontal>
+                        <samples>360</samples>
+                        <resolution>1</resolution>
+                        <min_angle>-3.14</min_angle>
+                        <max_angle>3.14</max_angle>
+                    </horizontal>
+                </scan>
+                <range>
+                    <min>0.2</min>
+                    <max>6</max>
+                    <resolution>0.05</resolution>
+                </range>
+                <noise>
+                    <type>gaussian</type>
+                    <mean>0.0</mean>
+                    <stddev>0.01</stddev>
+                </noise>
+            </ray>
+            <plugin name="laser" filename="libRayPlugin.so" />
+            <plugin name="gazebo_ros_head_rplidar_controller" filename="libgazebo_ros_laser.so">
+                <topicName>laser/scan</topicName>
+                <frameName>rplidar_link</frameName>
+            </plugin>
+            <always_on>1</always_on>
+            <update_rate>10</update_rate>
+            <visualize>true</visualize>
         </sensor>
     </gazebo>
@@ -61,33 +98,37 @@
         <plugin name="contactPlugin" filename="libunitreeFootContactPlugin.so"/>
         <contact>
-            <collision>FR_calf_fixed_joint_lump__FR_foot_collision_1</collision>
-        </contact>
+            <collision>
+                    FR_calf_fixed_joint_lump__FR_foot_collision_1</collision>
+            </contact>
         </sensor>
     </gazebo>
     <gazebo reference="FL_calf">
         <sensor name="FL_foot_contact" type="contact">
-        <update_rate>100</update_rate>
+        <update_rate>
+                100</update_rate>
         <plugin name="contactPlugin" filename="libunitreeFootContactPlugin.so"/>
         <contact>
             <collision>FL_calf_fixed_joint_lump__FL_foot_collision_1</collision>
-        </contact>
+            </contact>
         </sensor>
     </gazebo>
     <gazebo reference="RR_calf">
         <sensor name="RR_foot_contact" type="contact">
-        <update_rate>100</update_rate>
+        <update_rate>
+                100</update_rate>
         <plugin name="contactPlugin" filename="libunitreeFootContactPlugin.so"/>
         <contact>
             <collision>RR_calf_fixed_joint_lump__RR_foot_collision_1</collision>
-        </contact>
+            </contact>
         </sensor>
     </gazebo>
     <gazebo reference="RL_calf">
         <sensor name="RL_foot_contact" type="contact">
-        <update_rate>100</update_rate>
+        <update_rate>
+                100</update_rate>
         <plugin name="contactPlugin" filename="libunitreeFootContactPlugin.so"/>
         <contact>
             <collision>RL_calf_fixed_joint_lump__RL_foot_collision_1</collision>
-        </contact>
+            </contact>
         </sensor>
     </gazebo>
@@ -96,5 +137,6 @@
         <visual>
             <plugin name="drawForcePlugin" filename="libunitreeDrawForcePlugin.so">
-                <topicName>FR_foot_contact</topicName>
+                <topicName>
+                    FR_foot_contact</topicName>
             </plugin>
         </visual>
@@ -103,5 +145,6 @@
         <visual>
             <plugin name="drawForcePlugin" filename="libunitreeDrawForcePlugin.so">
-                <topicName>FL_foot_contact</topicName>
+                <topicName>
+                    FL_foot_contact</topicName>
             </plugin>
         </visual>
@@ -110,5 +153,6 @@
         <visual>
             <plugin name="drawForcePlugin" filename="libunitreeDrawForcePlugin.so">
-                <topicName>RR_foot_contact</topicName>
+                <topicName>
+                    RR_foot_contact</topicName>
             </plugin>
         </visual>
@@ -117,10 +161,12 @@
         <visual>
             <plugin name="drawForcePlugin" filename="libunitreeDrawForcePlugin.so">
-                <topicName>RL_foot_contact</topicName>
+                <topicName>
+                    RL_foot_contact</topicName>
             </plugin>
         </visual>
     </gazebo>
     <gazebo reference="base">
-        <material>Gazebo/Green</material>
+        <material>
+            Gazebo/Green</material>
         <turnGravityOff>false</turnGravityOff>
     </gazebo>
@@ -132,5 +178,6 @@
     </gazebo>
     <gazebo reference="stick_link">
-        <mu1>0.2</mu1>
+        <mu1>
+            0.2</mu1>
         <mu2>0.2</mu2>
         <material>Gazebo/White</material>
@@ -143,5 +190,6 @@
     <!-- FL leg -->
     <gazebo reference="FL_hip">
-        <mu1>0.2</mu1>
+        <mu1>
+            0.2</mu1>
         <mu2>0.2</mu2>
         <material>Gazebo/DarkGrey</material>
@@ -151,5 +199,6 @@
         <mu2>0.2</mu2>
         <self_collide>1</self_collide>
-        <material>Gazebo/DarkGrey</material>
+        <material>
+            Gazebo/DarkGrey</material>
         <kp  value="1000000.0"/>
         <kd  value="1.0"/>
@@ -161,5 +210,6 @@
     </gazebo>
     <gazebo reference="FL_foot">
-        <mu1>0.6</mu1>
+        <mu1>
+            0.6</mu1>
         <mu2>0.6</mu2>
         <self_collide>1</self_collide>
@@ -172,5 +222,6 @@
         <mu1>0.2</mu1>
         <mu2>0.2</mu2>
-        <material>Gazebo/DarkGrey</material>
+        <material>
+            Gazebo/DarkGrey</material>
     </gazebo>
     <gazebo reference="FR_thigh">
@@ -183,5 +234,6 @@
     </gazebo>
     <gazebo reference="FR_calf">
-        <mu1>0.2</mu1>
+        <mu1>
+            0.2</mu1>
         <mu2>0.2</mu2>
         <self_collide>1</self_collide>
@@ -191,5 +243,6 @@
         <mu2>0.6</mu2>
         <self_collide>1</self_collide>
-        <material>Gazebo/DarkGrey</material>
+        <material>
+            Gazebo/DarkGrey</material>
         <kp  value="1000000.0"/>
         <kd  value="1.0"/>
@@ -202,5 +255,6 @@
     </gazebo>
     <gazebo reference="RL_thigh">
-        <mu1>0.2</mu1>
+        <mu1>
+            0.2</mu1>
         <mu2>0.2</mu2>
         <self_collide>1</self_collide>
@@ -212,5 +266,6 @@
         <mu1>0.2</mu1>
         <mu2>0.2</mu2>
-        <self_collide>1</self_collide>
+        <self_collide>
+            1</self_collide>
     </gazebo>
     <gazebo reference="RL_foot">
@@ -224,5 +279,6 @@
     <!-- RR leg -->
     <gazebo reference="RR_hip">
-        <mu1>0.2</mu1>
+        <mu1>
+            0.2</mu1>
         <mu2>0.2</mu2>
         <material>Gazebo/DarkGrey</material>
@@ -232,5 +288,6 @@
         <mu2>0.2</mu2>
         <self_collide>1</self_collide>
-        <material>Gazebo/DarkGrey</material>
+        <material>
+            Gazebo/DarkGrey</material>
         <kp  value="1000000.0"/>
         <kd  value="1.0"/>
@@ -242,5 +299,6 @@
     </gazebo>
     <gazebo reference="RR_foot">
-        <mu1>0.6</mu1>
+        <mu1>
+            0.6</mu1>
         <mu2>0.6</mu2>
         <self_collide>1</self_collide>

File: robots/laikago_description/xacro/robot.xacro (robot description, xacro)
@@ -1,27 +1,52 @@
 <?xml version="1.0"?>
 <robot name="laikago" xmlns:xacro="http://www.ros.org/wiki/xacro">
-    <xacro:arg name="DEBUG" default="false"/>
-    <xacro:include filename="$(find laikago_description)/xacro/const.xacro"/>
-    <xacro:include filename="$(find laikago_description)/xacro/materials.xacro"/>
-    <xacro:include filename="$(find laikago_description)/xacro/leg.xacro"/>
-    <xacro:include filename="$(find laikago_description)/xacro/gazebo.xacro"/>
+    <xacro:arg name="DEBUG" default="false" />
+    <xacro:include filename="$(find laikago_description)/xacro/const.xacro" />
+    <xacro:include filename="$(find laikago_description)/xacro/materials.xacro" />
+    <xacro:include filename="$(find laikago_description)/xacro/leg.xacro" />
+    <xacro:include filename="$(find laikago_description)/xacro/gazebo.xacro" />
     <!-- Rollover Protection mode will add an additional stick on the top, use "true" or "false" to switch it. -->
-    <xacro:property name="rolloverProtection" value="false"/>
+    <xacro:property name="rolloverProtection" value="false" />
     <!-- Debug mode will hung up the robot, use "true" or "false" to switch it. -->
     <xacro:if value="$(arg DEBUG)">
-        <link name="world"/>
+        <link name="world" />
         <joint name="base_static_joint" type="fixed">
-            <origin rpy="0 0 0" xyz="0 0 0"/>
-            <parent link="world"/>
-            <child link="base"/>
+            <origin rpy="0 0 0" xyz="0 0 0" />
+            <parent link="world" />
+            <child link="base" />
         </joint>
     </xacro:if>
     <link name="base">
         <visual>
-            <origin rpy="0 0 0" xyz="0 0 0"/>
+            <origin rpy="0 0 0" xyz="0 0 0" />
             <geometry>
-                <box size="0.001 0.001 0.001"/>
+                <box size="0.001 0.001 0.001" />
             </geometry>
         </visual>
+    </link>
+    <joint name='lidar_joint' type='fixed'>
+        <parent link="base" />
+        <child link="lidar_link" />
+        <origin rpy="0 0 0" xyz="0 0 0.15" />
+    </joint>
+    <link name='lidar_link'>
+        <inertial>
+            <mass value="0.001" />
+            <origin rpy="0 0 0" xyz="0 0 0" />
+            <inertia ixx="0.0001" ixy="0" ixz="0" iyy="0.0001" iyz="0" izz="0.0001" />
+        </inertial>
+        <visual>
+            <origin rpy="0 0 0" xyz="0 0 0" />
+            <geometry>
+                <box size="0.001 0.001 0.001" />
+            </geometry>
+            <material name="red" />
+        </visual>
+        <collision>
+            <origin rpy="0 0 0" xyz="0 0 0" />
+            <geometry>
+                <box size=".001 .001 .001" />
+            </geometry>
+        </collision>
     </link>
     <joint name="floating_base" type="fixed">
